File: FliperKAd/FliperKAd.kicad_pcb (KiCad board)
At the start: 2 copper layers, 26 parts, among them J1 Conn_01x02, J2 Conn_ST_STDC14, J5 Conn_01x02, U1 STM32G431KBTx, U3 MCP1640x-xMC

Commit message: PCB Routé
Parts:
- added JP1: SolderJumper_2_Open, Jumper:SolderJumper-2_P1.3mm_Open_TrianglePad1.0x1.5mm, F.Cu at (223.8, 78.2)
- moved H3 102.1 mm to (221.0, 100.2)
- moved H2 100.3 mm to (221.0, 66.9)
- moved C3 90.4 mm to (221.8, 93.5)
- moved D1 87.7 mm to (213.0, 72.0), turned to -90 degrees
- moved J5 86.3 mm to (208.5, 103.2)
- moved C2 86.0 mm to (217.5, 89.8), turned to -90 degrees
- moved TP2 83.8 mm to (226.8, 81.3)
- moved C4 83.3 mm to (217.5, 85.2), turned to -90 degrees
- moved R5 82.1 mm to (219.0, 95.0), turned to -90 degrees
- moved J1 81.7 mm to (210.0, 62.9), turned to 180 degrees
- moved R3 81.5 mm to (217.5, 92.8), turned to -90 degrees
- moved C6 80.8 mm to (216.5, 79.0), turned to -90 degrees
- moved L2 80.6 mm to (219.2, 77.5), turned to 90 degrees
- moved H4 78.5 mm to (198.4, 100.2)
- moved H1 77.6 mm to (198.4, 66.9)
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Connections:
- C4 pad 1: +3.3V -> /Test 3.3
- R4 pad 1: +3.3V -> /Test 3.3
- TP2 pad 1: +3.3V -> /Test 3.3
- U3 pad 6: +3.3V -> /Test 3.3
- U3 pad 7: +3.3V -> /Test 3.3
Routing:
- net +3.3V: track 0.00 -> 51.9 mm, vias 0 -> 2
- net GND: track 0.00 -> 51.4 mm, vias 0 -> 55
- net +24V: track 0.00 -> 26.6 mm
- net Net-(U3-FB): track 0.00 -> 22.2 mm
- net USART2_RX: track 0.00 -> 21.8 mm
- net /Test 3.3: track 0.00 -> 17.1 mm
- net USART2_TX: track 0.00 -> 16.6 mm
- net NRST: track 0.00 -> 14.9 mm
- net Bouton_Actif: track 0.00 -> 13.4 mm
- net SYS_SWDIO: track 0.00 -> 12.0 mm
- net SYS_SWCLK: track 0.00 -> 9.95 mm
- net Net-(U3-EN): track 0.00 -> 7.54 mm, vias 0 -> 2
- net +3.3VA: track 0.00 -> 5.19 mm
- net Net-(U3-VCC): track 0.00 -> 4.25 mm
- net LED_Status: track 0.00 -> 3.45 mm
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- added copper zone on B.Cu, net GND
- added copper zone on F.Cu, net GND
Other:
- board outline added: 40 x 48.3 mm

Commit message: just in time
Parts:
- added D2: 1N4148WS, Diode_SMD:D_SOD-323, F.Cu at (185.0, 77.0)
- added D3: 1N4148WS, Diode_SMD:D_SOD-323, F.Cu at (185.0, 90.0)
- added J3: Conn_01x02, Connector_JST:JST_XH_B2B-XH-A_1x02_P2.50mm_Vertical, F.Cu at (181.0, 75.2)
- added J4: Conn_01x02, Connector_JST:JST_XH_B2B-XH-A_1x02_P2.50mm_Vertical, F.Cu at (181.0, 88.5)
- added Q1: NMOS, Package_TO_SOT_SMD:TO-263-3_TabPin4, F.Cu at (191.5, 104.7)
- added Q2: NMOS, Package_TO_SOT_SMD:TO-263-3_TabPin4, F.Cu at (205.0, 104.7)
- added R10: 4.7, Resistor_SMD:R_0603_1608Metric, F.Cu at (193.0, 71.0)
- added R11: 4.7, Resistor_SMD:R_0603_1608Metric, F.Cu at (193.0, 69.0)
- added R12: 10k, Resistor_SMD:R_0603_1608Metric, F.Cu at (190.0, 66.0)
- added R2: 10k, Resistor_SMD:R_0603_1608Metric, F.Cu at (225.0, 102.0)
- added R6: 10k, Resistor_SMD:R_0603_1608Metric, F.Cu at (222.0, 99.0)
- added R7: 10k, Resistor_SMD:R_0603_1608Metric, F.Cu at (200.0, 74.0)
- added R8: 10k, Resistor_SMD:R_0603_1608Metric, F.Cu at (208.0, 70.0)
- added R9: 10k, Resistor_SMD:R_0603_1608Metric, F.Cu at (192.0, 66.0)
- added U4: ~, Perso:MIC4426, F.Cu at (202.0, 69.0)
- moved H4 20.9 mm to (185.0, 116.2)
- moved TP1 17.4 mm to (221.0, 106.0)
- moved H3 16.0 mm to (221.0, 116.2)
- moved J5 16.0 mm to (208.5, 119.2)
- moved H1 13.4 mm to (185.0, 66.9)
Connections:
- U1 pad 20: unconnected-(U1-PA10-Pad20) -> Com-SolA
- U1 pad 21: unconnected-(U1-PA11-Pad21) -> Com-SolB
Routing:
- net +24V: track 26.6 -> 127.8 mm
- net Net-(Q1-G): track 0.00 -> 65.0 mm
- net +12V: track 0.00 -> 49.8 mm, vias 0 -> 2
- net Net-(Q2-G): track 0.00 -> 38.4 mm
- net Sortie-SolénoideB: track 0.00 -> 37.6 mm
- net Sortie-SolénoideA: track 0.00 -> 35.4 mm
- net Com-SolB: track 0.00 -> 17.5 mm
- net Com-SolA: track 0.00 -> 10.7 mm
- net Com-MOSB: track 0.00 -> 5.70 mm
- net Com-MOSA: track 0.00 -> 5.44 mm
- net GND: track 51.4 -> 53.3 mm, vias 55 -> 40
Other:
- board size 40 x 48.3 mm -> 53 x 64.2 mm

Commit message: pcb fini plus routage à valider et commander
Parts:
- removed R2, R6: 10k, Resistor_SMD:R_0603_1608Metric
- added C1: 100nF, Capacitor_SMD:C_0603_1608Metric, F.Cu at (226.2, 99.6)
- added C12: 10 µ, Capacitor_SMD:C_0603_1608Metric, F.Cu at (217.4, 97.6)
- added C5: 10 µ, Capacitor_SMD:C_0603_1608Metric, F.Cu at (217.4, 100.6)
- added JP2: SolderJumper_2_Open, Jumper:SolderJumper-2_P1.3mm_Open_TrianglePad1.0x1.5mm, F.Cu at (222.8, 100.2)
- added TP3: 12V, TestPoint:TestPoint_Pad_D2.0mm, F.Cu at (226.2, 97.2)
- added U5: ~, Perso:173951275, F.Cu at (223.6, 109.2)
- D2, D3: value 1N4148WS -> FSV340AF; footprint Diode_SMD:D_SOD-323 -> Diode_SMD:D_SMA
- moved TP1 18.2 mm to (210.4, 91.2)
- moved D2 0.80 mm to (185.8, 77.0)
- moved D3 0.80 mm to (185.8, 90.0)
Connections:
- U3 pad 12: Net-(U3-EN) -> +24V
- U3 pad 9: Net-(U3-EN) -> +24V
Routing:
- net +24V: track 127.8 -> 153.0 mm, vias 0 -> 3
- net Net-(U3-EN): track 7.54 -> 0.00 mm, vias 2 -> 0
- net /12test: track 0.00 -> 3.57 mm
- net GND: track 53.3 -> 55.0 mm, vias 40 -> 44
- net Net-(C12-Pad1): track 0.00 -> 1.45 mm
