File: FliperKAd/FliperKAd.kicad_pcb (KiCad board)
At the start: 2 copper layers, 53 x 64.2 mm, 46 parts, among them J1 Conn_01x02, J2 Conn_ST_STDC14, J3 Conn_01x02, J4 Conn_01x02, J5 Conn_01x02, Q1 NMOS, Q2 NMOS, U1 STM32G431KBTx, U3 MCP1640x-xMC

Commit message: dernière vérif avec Mr PPZ
Parts:
- Q1, Q2: footprint Package_TO_SOT_SMD:TO-263-3_TabPin4 -> Package_TO_SOT_SMD:TO-263-3_TabPin2
- moved C12 3.40 mm to (219.0, 100.6)
Connections:
- C12 pad 1: Net-(C12-Pad1) -> +24V
- C5 pad 2: Net-(C12-Pad1) -> GND
Routing:
- net Net-(Q1-G): track 65.0 -> 83.7 mm, vias 0 -> 2
- net Net-(Q2-G): track 38.4 -> 55.6 mm, vias 0 -> 2
- net GND: track 55.0 -> 59.3 mm
- net +24V: track 153.0 -> 154.6 mm
- net Net-(C12-Pad1): track 1.45 -> 0.00 mm
Other:
- board text added: "Driver Solénoide Flipper"
