File: FliperKAd/FliperKAd.kicad_sch (KiCad schematic)
At the start: 46 parts, among them J1 Conn_01x02, J2 Conn_ST_STDC14, J3 Conn_01x02, J4 Conn_01x02, J5 Conn_01x02, Q1 NMOS, Q2 NMOS, U1 STM32G431KBTx, U3 MCP1640x-xMC

Commit message: dernière vérif avec Mr PPZ
Parts:
- Q1, Q2: footprint Package_TO_SOT_SMD:TO-263-3_TabPin4 -> Package_TO_SOT_SMD:TO-263-3_TabPin2
Connections:
- net +24V: now also C12.1
- net GND: now also C5.2
Other:
- moved on the sheet: C12, C5
Changed lines of the file:
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@@
 	)
 	(junction
+		(at 115.57 154.94)
+		(diameter 0)
+		(color 0 0 0 0)
+	)
+	(junction
 		(at 97.79 31.75)
 		(diameter 0)
@@
 	(wire
 		(pts
-			(xy 115.57 153.67) (xy 115.57 154.94)
+			(xy 106.68 148.59) (xy 106.68 154.94)
 		)
 		(stroke
@@
 	(wire
 		(pts
+			(xy 106.68 142.24) (xy 106.68 143.51)
+		)
+		(stroke
+			(width 0)
+			(type default)
+		)
+	)
+	(wire
+		(pts
 			(xy 210.82 132.08) (xy 210.82 133.35)
 		)
@@
 	(wire
 		(pts
-			(xy 115.57 143.51) (xy 115.57 142.24)
+			(xy 115.57 146.05) (xy 115.57 142.24)
+		)
+		(stroke
+			(width 0)
+			(type default)
+		)
+	)
+	(wire
+		(pts
+			(xy 115.57 151.13) (xy 115.57 154.94)
 		)
 		(stroke
@@
 	(wire
 		(pts
-			(xy 115.57 154.94) (xy 127 154.94)
+			(xy 106.68 154.94) (xy 115.57 154.94)
 		)
 		(stroke
@@
 	(wire
 		(pts
+			(xy 115.57 154.94) (xy 127 154.94)
+		)
+		(stroke
+			(width 0)
+			(type default)
+		)
+	)
+	(wire
+		(pts
 			(xy 237.49 99.06) (xy 242.57 99.06)
 		)
@@
 	(wire
 		(pts
+			(xy 115.57 142.24) (xy 106.68 142.24)
+		)
+		(stroke
+			(width 0)
+			(type default)
+		)
+	)
+	(wire
+		(pts
 			(xy 210.82 55.88) (xy 212.09 55.88)
 		)
@@
 			)
 		)
-		(property "Footprint" "Package_TO_SOT_SMD:TO-263-3_TabPin4"
+		(property "Footprint" "Package_TO_SOT_SMD:TO-263-3_TabPin2"
 			(at 173.99 83.82 0)
 			(effects
@@
 	(symbol
 		(lib_id "Device:C_Small")
-		(at 115.57 151.13 0)
+		(at 106.68 146.05 0)
 		(unit 1)
 		(exclude_from_sim no)
@@
 		(fields_autoplaced yes)
 		(property "Reference" "C12"
-			(at 118.11 149.8662 0)
+			(at 109.22 144.7862 0)
 			(effects
 				(font
@@
 		)
 		(property "Value" "10 µ"
-			(at 118.11 152.4062 0)
+			(at 109.22 147.3262 0)
 			(effects
 				(font
@@
 		)
 		(property "Footprint" "Capacitor_SMD:C_0603_1608Metric"
-			(at 115.57 151.13 0)
+			(at 106.68 146.05 0)
 			(effects
 				(font
@@
 		)
 		(property "Datasheet" "~"
-			(at 115.57 151.13 0)
+			(at 106.68 146.05 0)
 			(effects
 				(font
@@
 		)
 		(property "Description" "Unpolarized capacitor, small symbol"
-			(at 115.57 151.13 0)
+			(at 106.68 146.05 0)
 			(effects
 				(font
@@
 			)
 		)
-		(property "Footprint" "Package_TO_SOT_SMD:TO-263-3_TabPin4"
+		(property "Footprint" "Package_TO_SOT_SMD:TO-263-3_TabPin2"
 			(at 173.99 36.83 0)
 			(effects
@@
 	(symbol
 		(lib_id "Device:C_Small")
-		(at 115.57 146.05 0)
+		(at 115.57 148.59 0)
 		(unit 1)
 		(exclude_from_sim no)
@@
 		(dnp no)
 		(property "Reference" "C5"
-			(at 108.966 143.764 0)
+			(at 108.966 146.304 0)
 			(effects
 				(font
@@
 		)
 		(property "Value" "10 µ"
-			(at 108.204 146.812 0)
+			(at 108.204 149.352 0)
 			(effects
 				(font
@@
 		)
 		(property "Footprint" "Capacitor_SMD:C_0603_1608Metric"
-			(at 115.57 146.05 0)
+			(at 115.57 148.59 0)
 			(effects
 				(font
@@
 		)
 		(property "Datasheet" "~"
-			(at 115.57 146.05 0)
+			(at 115.57 148.59 0)
 			(effects
 				(font
@@
 		)
 		(property "Description" "Unpolarized capacitor, small symbol"
-			(at 115.57 146.05 0)
+			(at 115.57 148.59 0)
 			(effects
 				(font
