File: hardware/FliperKAd/PCB_Final/Driver2Sol.kicad_sch (KiCad schematic)
At the start: 14 parts, among them J6 Conn_01x02, J7 Conn_01x02, Q10 NMOS, Q9 NMOS

Commit message: reset PCB final
Parts:
- added C202: 4u7, Capacitor_SMD:C_0603_1608Metric, symbol Device:C_Small
- C201: renamed from C16; value 100nF -> 100n
- J201: renamed from J7; footprint Connector_JST:JST_XH_B2B-XH-A_1x02_P2.50mm_Vertical -> Connector_JST:JST_PH_B2B-PH-K_1x02_P2.00mm_Vertical
- J202: renamed from J6; footprint Connector_JST:JST_XH_B2B-XH-A_1x02_P2.50mm_Vertical -> Connector_JST:JST_PH_B2B-PH-K_1x02_P2.00mm_Vertical
- R201: renamed from R30; value 4.7 -> 4R7; footprint Resistor_SMD:R_0603_1608Metric -> Resistor_SMD:R_0402_1005Metric
- R202: renamed from R31; footprint Resistor_SMD:R_0603_1608Metric -> Resistor_SMD:R_0402_1005Metric
- R203: renamed from R28; footprint Resistor_SMD:R_0603_1608Metric -> Resistor_SMD:R_0402_1005Metric
- R204: renamed from R29; footprint Resistor_SMD:R_0603_1608Metric -> Resistor_SMD:R_0402_1005Metric
- R205: renamed from R26; value 4.7 -> 4R7; footprint Resistor_SMD:R_0603_1608Metric -> Resistor_SMD:R_0402_1005Metric
- R206: renamed from R27; footprint Resistor_SMD:R_0603_1608Metric -> Resistor_SMD:R_0402_1005Metric
- U201: renamed from U9; value ~ -> MIC4427; MPN (none) -> MIC4427
- renumbered D5 to D201, D4 to D202, Q10 to Q201, Q9 to Q202
Connections:
- net GND: now also C202.2
- net 12V renamed +12V
- net +12V: now also C202.1
- net 24V renamed +24V
Other:
- moved on the sheet: C201, D201, D202, J201, J202, Q201, Q202, R201, R202, R203, R204, R205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
