File: hardware/FliperKAd/PCB_Final/PCB_Final.kicad_sch (KiCad schematic)
At the start: 34 parts, among them J1 Conn_01x02, J14 Conn_01x02, J15 Conn_01x10_MountingPin, J2 Conn_01x02, J3 Conn_01x02, J4 Conn_01x02, J5 Conn_ST_STDC14, U1 STM32G431KBTx

Commit message: reset PCB final
Parts:
- removed C12, C4, C8, C9: 10u, Capacitor_SMD:C_1206_3216Metric, symbol Device:C_Small
- removed C6: 100nF, Capacitor_SMD:C_0402_1005Metric, symbol Device:C_Small
- removed D3: LED_Small, LED_SMD:LED_0603_1608Metric, symbol Device:LED_Small
- removed J1, J14, J3, J4: Conn_01x02, Connector_JST:JST_XH_B2B-XH-A_1x02_P2.50mm_Vertical, symbol Connector_Generic:Conn_01x02
- removed J15: Conn_01x10_MountingPin, Perso:10pins, symbol Connector_Generic_MountingPin:Conn_01x10_MountingPin
- removed JP1, JP3: SolderJumper_2_Open, Jumper:SolderJumper-2_P1.3mm_Open_TrianglePad1.0x1.5mm, symbol Jumper:SolderJumper_2_Open
- removed TP1: 5V, TestPoint:TestPoint_Pad_D2.0mm, symbol Connector:TestPoint
- removed TP2: 3.3V, TestPoint:TestPoint_Pad_D2.0mm, symbol Connector:TestPoint
- removed U4, U5: ~, Perso:173951275, symbol Lib:173951275_
- added C107, C108, C109, C110: 10u, Capacitor_SMD:C_1206_3216Metric, symbol Device:C_Small
- added C111, C112: 1u, Capacitor_SMD:C_0603_1608Metric, symbol Device:C_Small
- added C113: 10n, Capacitor_SMD:C_0402_1005Metric, symbol Device:C_Small
- added C114: 100n, Capacitor_SMD:C_0402_1005Metric, symbol Device:C_Small
- added D101, D102, D103, D104, D105: LED, LED_SMD:LED_0603_1608Metric, symbol Device:LED
- added J103, J104: Conn_01x04, Connector_JST:JST_PH_B4B-PH-K_1x04_P2.00mm_Vertical, symbol Connector_Generic:Conn_01x04
- added J105: Conn_01x06, Connector_JST:JST_PH_B6B-PH-K_1x06_P2.00mm_Vertical, symbol Connector_Generic:Conn_01x06
- added J106: Conn_01x03, Connector_JST:JST_PH_B3B-PH-K_1x03_P2.00mm_Vertical, symbol Connector_Generic:Conn_01x03
- added JP102, JP103: SolderJumper_2_Open, Jumper:SolderJumper-2_P1.3mm_Open_TrianglePad1.0x1.5mm, symbol Jumper:SolderJumper_2_Open
- added R101: 22k3, Resistor_SMD:R_0402_1005Metric, symbol Device:R_Small
- added R102: 10k3, Resistor_SMD:R_0402_1005Metric, symbol Device:R_Small
- added R103: 3k3, Resistor_SMD:R_0402_1005Metric, symbol Device:R_Small
- added R104: 1k6, Resistor_SMD:R_0402_1005Metric, symbol Device:R_Small
- added R106, R109: 0R, Resistor_SMD:R_0402_1005Metric, symbol Device:R_Small
- added R107, R108, R110, R111, R112: 10k, Resistor_SMD:R_0402_1005Metric, symbol Device:R_Small
- added SW101, SW102, SW103: SW_Push, Maker:KSS221GLFS, symbol Switch:SW_Push
- added TP102: 5V, TestPoint:TestPoint_Pad_D2.0mm, symbol Connector:TestPoint
- added TP103: 3V3, TestPoint:TestPoint_Pad_D2.0mm, symbol Connector:TestPoint
- added U102, U103: ~, Perso:173951275, symbol Lib:173951275_
- C102: renamed from C2; value 100 nF -> 100n
- C103: renamed from C3; value 100 nF -> 100n
- C106: renamed from C5; value 10 nF -> 10n
- R105: renamed from R7; value 1k -> 1k7; footprint Resistor_SMD:R_0603_1608Metric -> Resistor_SMD:R_0402_1005Metric
- U101: renamed from U3; MPN (none) -> 173951275
- renumbered C1 to C101, C10 to C104, C11 to C105, H1 to H101, H2 to H102, H3 to H103, H4 to H104, J2 to J101, J5 to J102, JP2 to JP101, TP3 to TP101, U1 to U104
Connections:
- net +12V: now also R102.1
- net +24V: now also C107.1, C108.1, C109.1, C110.1, R101.1, U102.1 (Vin), U103.1 (Vin)
- net +3.3V: now also C112.1, J103.4 (Pin_4), J104.4 (Pin_4), J105.6 (Pin_6), JP103.2 (B), R104.1, R108.2, SW103.1
- net +5V: now also C111.1, J106.2 (Pin_2), JP102.2 (B), R103.1, R106.1, R109.1
- net Bouton_Droit: now also U104.6 (PA1), J103.3 (Pin_3), R107.1; no longer U104.31 (PB8)
- net Bouton_Gauche: now also J104.3 (Pin_3), R110.1
- net CS: now also J105.2 (Pin_2)
- net GND: now also C107.2, C108.2, C109.2, C110.2, C111.2, C112.2, C113.2, C114.2, D101.1 (K), D102.1 (K), D103.1 (K), D104.1 (K), J103.1 (Pin_1), J104.1 (Pin_1), J105.1 (Pin_1), J106.1 (Pin_1), R107.2, R110.2, R112.1, SW101.2, SW102.2, U102.2 (Gnd), U103.2 (Gnd)
- net LED_Stat: now also D105.1 (K)
- net LED_Status: now also D105.2 (A)
- net MISO: now also J105.4 (Pin_4)
- net MOSI: now also J105.5 (Pin_5)
- net NRST: now also C114.1, SW102.1
- net SCK: now also J105.3 (Pin_3)
- net TIM2: now also J106.3 (Pin_3)
- net USER_BTN: now reaches U104.22 (PA12)
- net USER_BTN: now also C113.1, R111.1
- net 12test: no longer names the net of JP101.1 (A), TP101.1, U101.3 (Vout)
- new net: J103.2 (Pin_2), R106.2
- new net: JP102.1 (A), TP102.1, U102.3 (Vout)
- new net: D104.2 (A), R104.2
- new net: J104.2 (Pin_2), R109.2
- new net: D103.2 (A), R103.2
- new net: D102.2 (A), R102.2
- new net: D101.2 (A), R101.2
- new net: R108.1, R111.2, SW101.1
- new net: JP103.1 (A), TP103.1, U103.3 (Vout)
- new net BOOT_0: R112.2, SW103.2, U104.31 (PB8)
- no-connect marks 9 -> 6
Other:
- sheet Driver 2 solénoïde renamed Driver 2 solénoïde 1
- removed sheet Driver 2 solénoïde1
- removed sheet Driver 2 solénoïde2
- removed sheet Driver 2 solénoïde3
- added sheet Driver 2 solénoïde 2 (Driver2Sol.kicad_sch)
- added sheet Driver 2 solénoïde 3 (Driver2Sol.kicad_sch)
- added sheet Driver 2 solénoïde 4 (Driver2Sol.kicad_sch)
- sheet Driver 2 solénoïde 1 ports: added none; removed 12V, 24V
- note added: "1mA @ 1.7V"
- note added: "Fixations"
- note added: "Gachettes"
- note added: "Interrupteurs"
- note added: "Neopixel"
- note added: "Photodiodes"
- note added: "Power Input"
- note added: "WPME 3V3"
- note removed: "WPME 3.3V"
- moved on the sheet: C101, C102, C103, C104, C105, C106, H101, H102, H103, H104, J101, J102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

Commit message: PCBogoss??
Parts:
- SW101, SW102, SW103: footprint Maker:KSS221GLFS -> Button_Switch_SMD:SW_SPST_B3U-3000P
Connections:
- net +5V: now also J106.3 (Pin_3); no longer J106.2 (Pin_2)
- net MOSI: now also J105.3 (Pin_3); no longer J105.5 (Pin_5)
- net SCK: now also J105.5 (Pin_5); no longer J105.3 (Pin_3)
- net TIM2: now also J106.2 (Pin_2); no longer J106.3 (Pin_3)

Commit message: pour le compte rendu
Parts:
- added J1, J2, J3: Conn_01x02, Connector_JST:JST_PH_B2B-PH-K_1x02_P2.00mm_Vertical, symbol Connector_Generic:Conn_01x02
Connections:
- net +3.3V: now also J3.2 (Pin_2)
- net GND: now also J1.1 (Pin_1), J2.1 (Pin_1), J3.1 (Pin_1)
- net Bump_Gauche: now reaches U104.2 (PF0)
- net Bump_Gauche: now also J2.2 (Pin_2)
- net Bump_Droit: now reaches U104.3 (PF1)
- net Bump_Droit: now also J1.2 (Pin_2)
- no-connect marks 6 -> 4
Other:
- note added: "Entrées solénoïdes"
- moved on the sheet: H101, H102, H103, H104
