File: hardware/FliperKAd/PCB_Final/PCB_Final.kicad_pcb (KiCad board)
At the start: 4 copper layers, 153 x 110 mm, 90 parts, among them J1 Conn_01x02, J10 Conn_01x02, J11 Conn_01x02, J12 Conn_01x02, J13 Conn_01x02, J14 Conn_01x02, J15 Conn_01x10_MountingPin, J2 Conn_01x02, J3 Conn_01x02, J4 Conn_01x02, J5 Conn_ST_STDC14, J6 Conn_01x02, J7 Conn_01x02, J8 Conn_01x02, J9 Conn_01x02, Q10 NMOS, Q11 NMOS, Q12 NMOS, Q13 NMOS, Q14 NMOS, Q15 NMOS, Q16 NMOS, Q9 NMOS, U1 STM32G431KBTx

Commit message: reset PCB final
Parts:
- removed C1: 4u7, Capacitor_SMD:C_0603_1608Metric
- removed C10, C11, C12, C4, C8, C9: 10u, Capacitor_SMD:C_1206_3216Metric
- removed C16, C17, C18, C19, C6: 100nF, Capacitor_SMD:C_0402_1005Metric
- removed C2, C3: 100 nF, Capacitor_SMD:C_0402_1005Metric
- removed C5: 10 nF, Capacitor_SMD:C_0402_1005Metric
- removed D10, D11, D4, D5, D6, D7, D8, D9: FSV340AF, Diode_SMD:D_SMA
- removed D3: LED_Small, LED_SMD:LED_0603_1608Metric
- removed H1, H2, H3, H4: MountingHole_Pad, MountingHole:MountingHole_3.2mm_M3_Pad_Via
- removed J1, J10, J11, J12, J13, J14, J3, J4, J6, J7, J8, J9: Conn_01x02, Connector_JST:JST_XH_B2B-XH-A_1x02_P2.50mm_Vertical
- removed J15: Conn_01x10_MountingPin, Perso:10pins
- removed J2: Conn_01x02, Connector_AMASS:AMASS_XT30U-F_1x02_P5.0mm_Vertical
- removed J5: Conn_ST_STDC14, Connector_PinHeader_1.27mm:PinHeader_2x07_P1.27mm_Vertical_SMD
- removed JP1, JP2, JP3: SolderJumper_2_Open, Jumper:SolderJumper-2_P1.3mm_Open_TrianglePad1.0x1.5mm
- removed Q10, Q11, Q12, Q13, Q14, Q15, Q16, Q9: NMOS, Perso:BUK
- removed R26, R30, R34, R36, R40, R42, R46, R48: 4.7, Resistor_SMD:R_0603_1608Metric
- removed R27, R28, R29, R31, R32, R33, R35, R37, R38, R39, R41, R43, R44, R45, R47, R49: 10k, Resistor_SMD:R_0603_1608Metric
- removed R7: 1k, Resistor_SMD:R_0603_1608Metric
- removed TP1: 5V, TestPoint:TestPoint_Pad_D2.0mm
- removed TP2: 3.3V, TestPoint:TestPoint_Pad_D2.0mm
- removed TP3: 12V, TestPoint:TestPoint_Pad_D2.0mm
- removed U1: STM32G431KBTx, Package_QFP:LQFP-32_7x7mm_P0.8mm
- removed U10, U11, U12, U9: ~, Package_SO:SOIC-8_5.3x6.2mm_P1.27mm
- removed U3, U4, U5: ~, Perso:173951275
- added C101: 4u7, Capacitor_SMD:C_0603_1608Metric, F.Cu at (185.0, 79.8)
- added C102: 100n, Capacitor_SMD:C_0402_1005Metric, F.Cu at (207.1, 75.8)
- added C103: 100n, Capacitor_SMD:C_0402_1005Metric, F.Cu at (207.1, 77.8)
- added C104: 10u, Capacitor_SMD:C_1206_3216Metric, F.Cu at (180.2, 49.6)
- added C105: 10u, Capacitor_SMD:C_1206_3216Metric, F.Cu at (180.2, 52.9)
- added C106: 10n, Capacitor_SMD:C_0402_1005Metric, F.Cu at (207.1, 79.7)
- added C107: 10u, Capacitor_SMD:C_1206_3216Metric, F.Cu at (180.2, 56.3)
- added C108: 10u, Capacitor_SMD:C_1206_3216Metric, F.Cu at (180.2, 59.6)
- added C109: 10u, Capacitor_SMD:C_1206_3216Metric, F.Cu at (180.2, 63.0)
- added C110: 10u, Capacitor_SMD:C_1206_3216Metric, F.Cu at (180.2, 66.3)
- added C111: 1u, Capacitor_SMD:C_0603_1608Metric, F.Cu at (185.0, 82.3)
- added C112: 1u, Capacitor_SMD:C_0603_1608Metric, F.Cu at (185.0, 84.8)
- added C113: 10n, Capacitor_SMD:C_0402_1005Metric, F.Cu at (207.1, 81.7)
- added C114: 100n, Capacitor_SMD:C_0402_1005Metric, F.Cu at (207.1, 83.7)
- added C201: 100n, Capacitor_SMD:C_0402_1005Metric, F.Cu at (224.7, 105.9)
- added C202: 4u7, Capacitor_SMD:C_0603_1608Metric, F.Cu at (221.2, 106.1)
- added C301: 100n, Capacitor_SMD:C_0402_1005Metric, F.Cu at (225.8, 65.7)
- added C302: 4u7, Capacitor_SMD:C_0603_1608Metric, F.Cu at (222.3, 66.0)
- added C401: 100n, Capacitor_SMD:C_0402_1005Metric, F.Cu at (203.7, 105.9)
- added C402: 4u7, Capacitor_SMD:C_0603_1608Metric, F.Cu at (200.3, 106.1)
- added C501: 100n, Capacitor_SMD:C_0402_1005Metric, F.Cu at (182.8, 105.9)
- added C502: 4u7, Capacitor_SMD:C_0603_1608Metric, F.Cu at (179.3, 106.1)
- added D101: LED, LED_SMD:LED_0603_1608Metric, F.Cu at (208.4, 49.2)
- added D102: LED, LED_SMD:LED_0603_1608Metric, F.Cu at (208.4, 51.8)
- added D103: LED, LED_SMD:LED_0603_1608Metric, F.Cu at (208.4, 54.4)
- added D104: LED, LED_SMD:LED_0603_1608Metric, F.Cu at (208.4, 57.0)
- added D105: LED, LED_SMD:LED_0603_1608Metric, F.Cu at (208.4, 59.6)
- added D201: FSV340AF, Diode_SMD:D_SMA, F.Cu at (223.3, 98.1)
- added D202: FSV340AF, Diode_SMD:D_SMA, F.Cu at (223.3, 102.6)
- added D301: FSV340AF, Diode_SMD:D_SMA, F.Cu at (224.4, 57.9)
- added D302: FSV340AF, Diode_SMD:D_SMA, F.Cu at (224.4, 62.5)
- added D401: FSV340AF, Diode_SMD:D_SMA, F.Cu at (202.3, 98.1)
- added D402: FSV340AF, Diode_SMD:D_SMA, F.Cu at (202.3, 102.6)
- added D501: FSV340AF, Diode_SMD:D_SMA, F.Cu at (181.4, 98.1)
- added D502: FSV340AF, Diode_SMD:D_SMA, F.Cu at (181.4, 102.6)
- added H101: MountingHole_Pad, MountingHole:MountingHole_3.2mm_M3_Pad_Via, F.Cu at (55.0, 55.0)
- added H102: MountingHole_Pad, MountingHole:MountingHole_3.2mm_M3_Pad_Via, F.Cu at (125.0, 55.0)
- added H103: MountingHole_Pad, MountingHole:MountingHole_3.2mm_M3_Pad_Via, F.Cu at (55.0, 125.0)
- added H104: MountingHole_Pad, MountingHole:MountingHole_3.2mm_M3_Pad_Via, F.Cu at (125.0, 125.0)
- added J101: Conn_01x02, Connector_AMASS:AMASS_XT30U-F_1x02_P5.0mm_Vertical, F.Cu at (196.2, 71.2)
- added J102: Conn_ST_STDC14, Connector_PinHeader_1.27mm:PinHeader_2x07_P1.27mm_Vertical_SMD, F.Cu at (187.8, 73.0)
- added J103: Conn_01x04, Connector_JST:JST_PH_B4B-PH-K_1x04_P2.00mm_Vertical, F.Cu at (185.9, 50.6)
- added J104: Conn_01x04, Connector_JST:JST_PH_B4B-PH-K_1x04_P2.00mm_Vertical, F.Cu at (185.9, 57.2)
- added J105: Conn_01x06, Connector_JST:JST_PH_B6B-PH-K_1x06_P2.00mm_Vertical, F.Cu at (185.9, 63.7)
- added J106: Conn_01x03, Connector_JST:JST_PH_B3B-PH-K_1x03_P2.00mm_Vertical, F.Cu at (201.9, 63.7)
- added J201: Conn_01x02, Connector_JST:JST_PH_B2B-PH-K_1x02_P2.00mm_Vertical, F.Cu at (214.2, 90.8)
- added J202: Conn_01x02, Connector_JST:JST_PH_B2B-PH-K_1x02_P2.00mm_Vertical, F.Cu at (214.2, 97.3)
- added J301: Conn_01x02, Connector_JST:JST_PH_B2B-PH-K_1x02_P2.00mm_Vertical, F.Cu at (215.4, 50.6)
- added J302: Conn_01x02, Connector_JST:JST_PH_B2B-PH-K_1x02_P2.00mm_Vertical, F.Cu at (215.4, 57.2)
- added J401: Conn_01x02, Connector_JST:JST_PH_B2B-PH-K_1x02_P2.00mm_Vertical, F.Cu at (193.3, 90.8)
- added J402: Conn_01x02, Connector_JST:JST_PH_B2B-PH-K_1x02_P2.00mm_Vertical, F.Cu at (193.3, 97.3)
- added J501: Conn_01x02, Connector_JST:JST_PH_B2B-PH-K_1x02_P2.00mm_Vertical, F.Cu at (172.3, 90.8)
- added J502: Conn_01x02, Connector_JST:JST_PH_B2B-PH-K_1x02_P2.00mm_Vertical, F.Cu at (172.3, 97.3)
- added JP101: SolderJumper_2_Open, Jumper:SolderJumper-2_P1.3mm_Open_TrianglePad1.0x1.5mm, F.Cu at (203.5, 76.6)
- added JP102: SolderJumper_2_Open, Jumper:SolderJumper-2_P1.3mm_Open_TrianglePad1.0x1.5mm, F.Cu at (203.5, 80.1)
- added JP103: SolderJumper_2_Open, Jumper:SolderJumper-2_P1.3mm_Open_TrianglePad1.0x1.5mm, F.Cu at (203.5, 83.7)
- added R101: 22k3, Resistor_SMD:R_0402_1005Metric, F.Cu at (194.1, 75.8)
- added R102: 10k3, Resistor_SMD:R_0402_1005Metric, F.Cu at (194.1, 77.8)
- added R103: 3k3, Resistor_SMD:R_0402_1005Metric, F.Cu at (194.1, 79.8)
- added R104: 1k6, Resistor_SMD:R_0402_1005Metric, F.Cu at (194.1, 81.8)
- added R105: 1k7, Resistor_SMD:R_0402_1005Metric, F.Cu at (197.0, 75.8)
- added R106: 0R, Resistor_SMD:R_0402_1005Metric, F.Cu at (197.0, 77.8)
- added R107: 10k, Resistor_SMD:R_0402_1005Metric, F.Cu at (197.0, 79.8)
- added R108: 10k, Resistor_SMD:R_0402_1005Metric, F.Cu at (197.0, 81.8)
- added R109: 0R, Resistor_SMD:R_0402_1005Metric, F.Cu at (199.9, 75.8)
- added R110: 10k, Resistor_SMD:R_0402_1005Metric, F.Cu at (199.9, 77.8)
- added R111: 10k, Resistor_SMD:R_0402_1005Metric, F.Cu at (199.9, 79.8)
- added R112: 10k, Resistor_SMD:R_0402_1005Metric, F.Cu at (199.9, 81.8)
- added R201: 4R7, Resistor_SMD:R_0402_1005Metric, F.Cu at (228.8, 96.8)
- added R202: 10k, Resistor_SMD:R_0402_1005Metric, F.Cu at (228.8, 98.8)
- added R203: 10k, Resistor_SMD:R_0402_1005Metric, F.Cu at (228.8, 100.8)
- added R204: 10k, Resistor_SMD:R_0402_1005Metric, F.Cu at (228.8, 102.7)
- added R205: 4R7, Resistor_SMD:R_0402_1005Metric, F.Cu at (228.8, 104.7)
- added R206: 10k, Resistor_SMD:R_0402_1005Metric, F.Cu at (228.8, 106.7)
- added R301: 4R7, Resistor_SMD:R_0402_1005Metric, F.Cu at (229.9, 56.6)
- added R302: 10k, Resistor_SMD:R_0402_1005Metric, F.Cu at (229.9, 58.6)
- added R303: 10k, Resistor_SMD:R_0402_1005Metric, F.Cu at (229.9, 60.6)
- added R304: 10k, Resistor_SMD:R_0402_1005Metric, F.Cu at (229.9, 62.6)
- added R305: 4R7, Resistor_SMD:R_0402_1005Metric, F.Cu at (229.9, 64.6)
- added R306: 10k, Resistor_SMD:R_0402_1005Metric, F.Cu at (229.9, 66.6)
- added R401: 4R7, Resistor_SMD:R_0402_1005Metric, F.Cu at (207.8, 96.8)
- added R402: 10k, Resistor_SMD:R_0402_1005Metric, F.Cu at (207.8, 98.8)
- added R403: 10k, Resistor_SMD:R_0402_1005Metric, F.Cu at (207.8, 100.8)
- added R404: 10k, Resistor_SMD:R_0402_1005Metric, F.Cu at (207.8, 102.7)
- added R405: 4R7, Resistor_SMD:R_0402_1005Metric, F.Cu at (207.8, 104.7)
- added R406: 10k, Resistor_SMD:R_0402_1005Metric, F.Cu at (207.8, 106.7)
- added R501: 4R7, Resistor_SMD:R_0402_1005Metric, F.Cu at (186.9, 96.8)
- added R502: 10k, Resistor_SMD:R_0402_1005Metric, F.Cu at (186.9, 98.8)
- added R503: 10k, Resistor_SMD:R_0402_1005Metric, F.Cu at (186.9, 100.8)
- added R504: 10k, Resistor_SMD:R_0402_1005Metric, F.Cu at (186.9, 102.7)
- added R505: 4R7, Resistor_SMD:R_0402_1005Metric, F.Cu at (186.9, 104.7)
- added R506: 10k, Resistor_SMD:R_0402_1005Metric, F.Cu at (186.9, 106.7)
- added TP101: 12V, TestPoint:TestPoint_Pad_D2.0mm, F.Cu at (179.3, 70.0)
- added TP102: 5V, TestPoint:TestPoint_Pad_D2.0mm, F.Cu at (179.3, 74.1)
- added TP103: 3V3, TestPoint:TestPoint_Pad_D2.0mm, F.Cu at (179.3, 78.1)
- added U104: STM32G431KBTx, Package_QFP:LQFP-32_7x7mm_P0.8mm, F.Cu at (200.6, 53.6)
- added U201: MIC4427, Package_SO:SOIC-8_5.3x6.2mm_P1.27mm, F.Cu at (224.4, 91.9)
- added U301: MIC4427, Package_SO:SOIC-8_5.3x6.2mm_P1.27mm, F.Cu at (225.6, 51.8)
- added U401: MIC4427, Package_SO:SOIC-8_5.3x6.2mm_P1.27mm, F.Cu at (203.5, 91.9)
- added U501: MIC4427, Package_SO:SOIC-8_5.3x6.2mm_P1.27mm, F.Cu at (182.6, 91.9)
Routing:
- net +3.3V: track 246.7 -> 0.00 mm
- net +24V: track 93.8 -> 0.00 mm
- net Bouton_Droit: track 79.1 -> 0.00 mm, vias 2 -> 0
- net TIM2: track 76.5 -> 0.00 mm, vias 2 -> 0
- net GND: track 70.7 -> 0.00 mm, vias 11 -> 0
- net MOSI: track 69.0 -> 0.00 mm, vias 2 -> 0
- net SCK: track 68.1 -> 0.00 mm, vias 2 -> 0
- net MISO: track 57.0 -> 0.00 mm, vias 2 -> 0
- net CS: track 56.6 -> 0.00 mm, vias 2 -> 0
- net Com-SolH: track 53.6 -> 0.00 mm
- net Com-SolA: track 53.0 -> 0.00 mm
- net Com-SolG: track 52.4 -> 0.00 mm
- net Bouton_Gauche: track 51.7 -> 0.00 mm, vias 2 -> 0
- net Com-SolB: track 49.1 -> 0.00 mm
- net /5test: track 47.3 -> 0.00 mm
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- added copper zone on B.Cu, net GND
- removed copper zone on In2.Cu, net +12V
- removed copper zone on B.Cu, net +24V
- removed copper zone on F.Cu, net +24V
- removed copper zone on In1.Cu, net +5V
- removed copper zone on F.Cu, net Net-(D10-A)
- removed copper zone on F.Cu, net Net-(D11-A)
- removed copper zone on F.Cu, net Net-(D4-A)
- removed copper zone on F.Cu, net Net-(D5-A)
- removed copper zone on F.Cu, net Net-(D6-A)
- removed copper zone on F.Cu, net Net-(D7-A)
- removed copper zone on F.Cu, net Net-(D8-A)
- removed copper zone on F.Cu, net Net-(D9-A)
Other:
- board size 153 x 110 mm -> 80 x 80 mm

Commit message: PCBogoss??
Parts:
- added Q201: NMOS, Perso:BUK, F.Cu at (60.0, 121.0)
- added Q202: NMOS, Perso:BUK, F.Cu at (47.7, 121.0)
- added Q301: NMOS, Perso:BUK, F.Cu at (84.3, 121.1)
- added Q302: NMOS, Perso:BUK, F.Cu at (72.2, 121.1)
- added Q401: NMOS, Perso:BUK, F.Cu at (108.2, 121.1)
- added Q402: NMOS, Perso:BUK, F.Cu at (96.3, 121.1)
- added Q501: NMOS, Perso:BUK, F.Cu at (132.5, 121.1)
- added Q502: NMOS, Perso:BUK, F.Cu at (120.2, 121.1)
- added SW101: SW_Push, Button_Switch_SMD:SW_SPST_B3U-3000P, F.Cu at (86.0, 98.7)
- added SW102: SW_Push, Button_Switch_SMD:SW_SPST_B3U-3000P, F.Cu at (62.8, 75.3)
- added SW103: SW_Push, Button_Switch_SMD:SW_SPST_B3U-3000P, F.Cu at (98.5, 92.0)
- added U101: ~, Perso:173951275, F.Cu at (101.2, 49.5)
- added U102: ~, Perso:173951275, F.Cu at (85.9, 49.5)
- added U103: ~, Perso:173951275, F.Cu at (70.9, 49.5)
- moved R206 179.0 mm to (49.8, 108.5), turned to 180 degrees
- moved R204 179.0 mm to (50.0, 94.0), turned to 180 degrees
- moved R205 178.5 mm to (50.2, 106.0), turned to 90 degrees
- moved R203 175.4 mm to (53.5, 94.0)
- moved R304 174.2 mm to (58.5, 94.0), turned to 180 degrees
- moved D202 173.5 mm to (52.0, 130.0), turned to 180 degrees
- moved U201 172.2 mm to (52.4, 99.5), turned to -90 degrees
- moved U301 171.5 mm to (60.8, 99.5), turned to -90 degrees
- moved R303 171.2 mm to (62.0, 94.0)
- moved C201 170.7 mm to (54.0, 108.0), turned to -90 degrees
- moved C202 168.7 mm to (52.5, 108.2), turned to -90 degrees
- moved R201 167.2 mm to (62.0, 108.5), turned to 180 degrees
- moved R202 167.1 mm to (62.0, 109.8), turned to 180 degrees
- moved J202 166.6 mm to (52.0, 135.0)
- moved D302 166.3 mm to (72.5, 130.2), turned to 180 degrees
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Connections:
- J105 pad 3: SCK -> MOSI
- J105 pad 5: MOSI -> SCK
- J106 pad 2: +5V -> TIM2
- J106 pad 3: TIM2 -> +5V
- R303 pad 1: Com-SolC -> Com-SolD
- R304 pad 1: Com-SolD -> Com-SolC
- R403 pad 1: Com-SolE -> Com-SolF
- R404 pad 1: Com-SolF -> Com-SolE
- R503 pad 1: Com-SolG -> Com-SolH
- R504 pad 1: Com-SolH -> Com-SolG
- U301 pad 2: Com-SolC -> Com-SolD
- U301 pad 4: Com-SolD -> Com-SolC
- U401 pad 2: Com-SolE -> Com-SolF
- U401 pad 4: Com-SolF -> Com-SolE
- U501 pad 2: Com-SolG -> Com-SolH
- U501 pad 4: Com-SolH -> Com-SolG
Routing:
- net +3.3V: track 0.00 -> 239.3 mm, vias 0 -> 1
- net +12V: track 0.00 -> 162.0 mm, vias 0 -> 7
- net MISO: track 0.00 -> 99.8 mm, vias 0 -> 1
- net SCK: track 0.00 -> 85.6 mm, vias 0 -> 1
- net MOSI: track 0.00 -> 77.4 mm, vias 0 -> 1
- net CS: track 0.00 -> 74.9 mm, vias 0 -> 2
- net Bouton_Gauche: track 0.00 -> 72.2 mm, vias 0 -> 2
- net +24V: track 0.00 -> 64.0 mm
- net Net-(U501-OUTA): track 0.00 -> 60.2 mm
- net +5V: track 0.00 -> 55.6 mm, vias 0 -> 5
- net Net-(U501-OUTB): track 0.00 -> 49.2 mm
- net Net-(U401-OUTA): track 0.00 -> 42.4 mm
- net /BOOT_0: track 0.00 -> 41.4 mm, vias 0 -> 2
- net Net-(U401-OUTB): track 0.00 -> 33.3 mm
- net USART2_RX: track 0.00 -> 32.5 mm, vias 0 -> 2
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- added copper zone on In1.Cu, net +12V
- added copper zone on F.Cu, net +24V
- added copper zone on In1.Cu, net +24V
- added copper zone on In1.Cu, net +5V
- added copper zone on In1.Cu, net GND
- added copper zone on In2.Cu, net GND
- added copper zone on F.Cu, net Net-(D201-A)
- added copper zone on F.Cu, net Net-(D202-A)
- added copper zone on F.Cu, net Net-(D301-A)
- added copper zone on F.Cu, net Net-(D302-A)
- added copper zone on F.Cu, net Net-(D401-A)
- added copper zone on F.Cu, net Net-(D402-A)
- added copper zone on F.Cu, net Net-(D501-A)
- added copper zone on F.Cu, net Net-(D502-A)
Other:
- board size 80 x 80 mm -> 100 x 100 mm

Commit message: personalisation
Parts:
- added G***: LOGO, LOGO, F.Cu at (52.5, 56.8)
Other:
- board text added: "Flipper_le_dauphin"

Commit message: pour le compte rendu
Parts:
- added J1: Conn_01x02, Connector_JST:JST_PH_B2B-PH-K_1x02_P2.00mm_Vertical, F.Cu at (43.5, 57.8)
- added J2: Conn_01x02, Connector_JST:JST_PH_B2B-PH-K_1x02_P2.00mm_Vertical, F.Cu at (43.5, 65.2)
- added J3: Conn_01x02, Connector_JST:JST_PH_B2B-PH-K_1x02_P2.00mm_Vertical, F.Cu at (124.0, 42.8)
Connections:
- U104 pad 2: unconnected-(U104-PF0-Pad2) -> Bump_Gauche
- U104 pad 3: unconnected-(U104-PF1-Pad3) -> Bump_Droit
Routing:
- net Bump_Droit: track 0.00 -> 36.3 mm, vias 0 -> 1
- net Bump_Gauche: track 0.00 -> 30.8 mm, vias 0 -> 1
- net +3.3V: track 239.3 -> 247.6 mm

Commit message: petit oubli'
Parts:
- moved U103 7.83 mm to (77.5, 53.8), turned to 180 degrees
- moved U101 7.79 mm to (107.6, 54.0), turned to 180 degrees
- moved U102 7.40 mm to (92.1, 53.7), turned to 180 degrees
Routing:
- net GND: track 23.3 -> 39.3 mm
- net +24V: track 64.0 -> 75.0 mm
- net Net-(JP102-A): track 17.9 -> 18.4 mm
